Commit message: Add URDF model for Otto robot with detailed links and joints
- Created a new URDF file for the Otto robot, defining its structure and components.
- Included links for the base, legs, feet, ultrasonic sensor, and head.
- Defined revolute joints for leg and foot movements, along with fixed joints for the ultrasonic sensor and body shell.
- Specified inertial properties, visual representations, and collision geometries for each link.

File: ros2_ws/src/otto_description/urdf/otto copy.urdf (robot description, URDF)
Before this commit: robot otto, 7 links, 6 joints
Links:
- removed link foot_left
- removed link foot_right
- removed link head
- removed link leg_left
- removed link leg_right
- removed link ultrasonic
- added link FootL_1, mass 0.01274684267714529; collision mesh filename=file:///ros2_ws/src/otto_description/meshes/foot_left.stl scale=0.001 0.001 0.001; visual mesh filename=file:///ros2_ws/src/otto_description/meshes/foot_left.stl scale=0.001 0.001 0.001
- added link FootR_1, mass 0.012749332366692666; collision mesh filename=file:///ros2_ws/src/otto_description/meshes/foot_right.stl scale=0.001 0.001 0.001; visual mesh filename=file:///ros2_ws/src/otto_description/meshes/foot_right.stl scale=0.001 0.001 0.001
- added link LeftLeg_1, mass 0.008295768110971864; collision mesh filename=file:///ros2_ws/src/otto_description/meshes/leg_left.stl scale=0.001 0.001 0.001; visual mesh filename=file:///ros2_ws/src/otto_description/meshes/leg_left.stl scale=0.001 0.001 0.001
- added link RightLeg_1, mass 0.00834817521109724; collision mesh filename=file:///ros2_ws/src/otto_description/meshes/leg_left.stl scale=0.001 0.001 0.001; visual mesh filename=file:///ros2_ws/src/otto_description/meshes/leg_left.stl scale=0.001 0.001 0.001
- added link Ultrasonic_Sensor_v1_1, mass 0.044351271100451166; collision mesh filename=file:///ros2_ws/src/otto_description/meshes/ultrasonic.stl scale=0.001 0.001 0.001; visual mesh filename=file:///ros2_ws/src/otto_description/meshes/ultrasonic.stl scale=0.001 0.001 0.001
- added link old_component__1__1, mass 0.0241983579475568; collision mesh filename=file:///ros2_ws/src/otto_description/meshes/head.stl scale=0.001 0.001 0.001; visual mesh filename=file:///ros2_ws/src/otto_description/meshes/head.stl scale=0.001 0.001 0.001
Joints:
- removed joint head_joint
- removed joint ultrasonic_joint
- added joint BodyShellJoint: type fixed, parent base_link, child old_component__1__1, origin xyz=0.033 0.0 -0.007 rpy=0 0 0
- added joint UltrasonicJoint: type fixed, parent base_link, child Ultrasonic_Sensor_v1_1, origin xyz=0.013675 -0.0327 0.0175 rpy=0 0 0
- joint LeftFoot: child foot_left -> FootL_1; parent leg_left -> LeftLeg_1
- joint LeftLeg: child leg_left -> LeftLeg_1
- joint RightFoot: child foot_right -> FootR_1; parent leg_right -> RightLeg_1
- joint RightLeg: child leg_right -> RightLeg_1
