Commit message: Add URDF and material files for Otto robot model
- Created fusion2urdf.txt to document URDF structure generated from Fusion Model.
- Added materials.xacro defining various materials used in the robot model.
- Introduced otto.xacro as the main URDF file for the Otto robot, including links and joints.
- Implemented otto_Descriptor_rev0.xacro with detailed specifications for each link and joint, including inertial properties and visual representations.
- Included Zone.Identifier files for metadata tracking.

File: ros2_ws/src/otto_description/urdf/otto_Descriptor_rev0.xacro (robot description, xacro)
@@ -2,6 +2,10 @@
 <robot xmlns:xacro="http://www.ros.org/wiki/xacro" name="otto">
    <xacro:include filename="$(find otto)/urdf/materials.xacro" />
-   <!-- ==================== LINKS ==================== -->
-   <link name="base_link">
+   <link name="dummy_link" />
+   <joint name="dummy_link_joint" type="fixed">
+      <parent link="dummy_link" />
+      <child link="base_link:1" />
+   </joint>
+   <link name="base_link_1">
       <inertial>
          <origin xyz="-0.017480908878091606 0.03519882134873651 -0.025083002755304264" rpy="0.0 0.0 0.0" />
@@ -234,30 +238,29 @@
       </collision>
    </link>
-   <!-- ==================== JOINTS ==================== -->
-   <joint name="leg_right_joint" type="revolute">
+   <joint name="Revolucionar46" type="revolute">
       <origin xyz="-0.012391174437753782 0.005158205912836682 -0.039" rpy="0.0 0.0 0.0" />
-      <parent link="base_link" />
+      <parent link="base_link_1" />
       <child link="RightLeg_1" />
       <axis xyz="0.0 0.0 1.0" />
       <limit upper="1.5707963267948966" lower="-1.5707963267948966" effort="100.0" velocity="100.0" />
    </joint>
-   <joint name="leg_left_joint" type="revolute">
+   <joint name="Revolucionar47" type="revolute">
       <origin xyz="-0.016999572875253794 0.061000427124746216 -0.037000000000000005" rpy="0.0 0.0 0.0" />
-      <parent link="base_link" />
+      <parent link="base_link_1" />
       <child link="LeftLeg_1" />
       <axis xyz="0.0 0.0 -1.0" />
       <limit upper="1.5707963267948966" lower="-1.5707963267948966" effort="100.0" velocity="100.0" />
    </joint>
-   <joint name="ultrasonic_joint" type="fixed">
+   <joint name="Gruporígido43" type="fixed">
       <origin xyz="0.0 0.0 0.0" rpy="0.0 0.0 0.0" />
-      <parent link="base_link" />
+      <parent link="base_link_1" />
       <child link="Ultrasonic_Sensor_v1_1_1" />
    </joint>
-   <joint name="head_joint" type="fixed">
+   <joint name="Gruporígido43_0" type="fixed">
       <origin xyz="0.00011642897127504436 6.011660760218973e-07 -0.0009665825749333657" rpy="0.0 0.0 0.0" />
-      <parent link="base_link" />
+      <parent link="base_link_1" />
       <child link="Head_1_1" />
    </joint>
-   <joint name="foot_right_joint" type="revolute">
+   <joint name="Revolucionar45" type="revolute">
       <origin xyz="0.0179 0.0 -0.031" rpy="0.0 0.0 0.0" />
       <parent link="RightLeg_1" />
@@ -266,5 +269,5 @@
       <limit upper="1.5707963267948966" lower="-1.5707963267948966" effort="100.0" velocity="100.0" />
    </joint>
-   <joint name="foot_left_joint" type="revolute">
+   <joint name="Revolucionar44" type="revolute">
       <origin xyz="0.0175 0.0 -0.031" rpy="0.0 0.0 0.0" />
       <parent link="LeftLeg_1" />
