Commit message: Enhance Otto's walking functionality and Gazebo integration
- Update commands for building and launching Otto in Gazebo.
- Adjust Gazebo launch parameters for improved robot positioning.
- Refactor Otto walking script to include joint position publishers and initial zero position setup.
- Add friction and damping properties to joints in the URDF for better simulation stability.

File: ros2_ws/src/otto_description/urdf/otto.xacro (robot description, xacro)
@@ -273,38 +273,87 @@
       <limit upper="1.5707963267948966" lower="-1.5707963267948966" effort="100.0" velocity="100.0" />
    </joint>
-   <!-- Plugin Gazebo para cada junta -->
-  <gazebo>
-    <plugin filename="gz-sim-joint-position-controller-system"
-            name="gz::sim::systems::JointPositionController">
-      <joint_name>leg_right_joint</joint_name>
-      <topic>/leg_right_joint/cmd</topic>
-      <p_gain>10</p_gain>
-      <i_gain>0</i_gain>
-      <d_gain>0.5</d_gain>
-    </plugin>
-    <plugin filename="gz-sim-joint-position-controller-system"
-            name="gz::sim::systems::JointPositionController">
-      <joint_name>leg_left_joint</joint_name>
-      <topic>/leg_left_joint/cmd</topic>
-      <p_gain>10</p_gain>
-      <i_gain>0</i_gain>
-      <d_gain>0.5</d_gain>
-    </plugin>
-    <plugin filename="gz-sim-joint-position-controller-system"
-            name="gz::sim::systems::JointPositionController">
-      <joint_name>foot_right_joint</joint_name>
-      <topic>/foot_right_joint/cmd</topic>
-      <p_gain>10</p_gain>
-      <i_gain>0</i_gain>
-      <d_gain>0.5</d_gain>
-    </plugin>
-    <plugin filename="gz-sim-joint-position-controller-system"
-            name="gz::sim::systems::JointPositionController">
-      <joint_name>foot_left_joint</joint_name>
-      <topic>/foot_left_joint/cmd</topic>
-      <p_gain>10</p_gain>
-      <i_gain>0</i_gain>
-      <d_gain>0.5</d_gain>
-    </plugin>
-  </gazebo>
+      <!-- Plugin Gazebo para cada junta -->
+   <gazebo>
+      <plugin filename="gz-sim-joint-position-controller-system"
+               name="gz::sim::systems::JointPositionController">
+         <joint_name>leg_right_joint</joint_name>
+         <topic>/leg_right_joint/cmd</topic>
+         <p_gain>20</p_gain>
+         <i_gain>0</i_gain>
+         <d_gain>2.0</d_gain>
+      </plugin>
+      <plugin filename="gz-sim-joint-position-controller-system"
+               name="gz::sim::systems::JointPositionController">
+         <joint_name>leg_left_joint</joint_name>
+         <topic>/leg_left_joint/cmd</topic>
+         <p_gain>20</p_gain>
+         <i_gain>0</i_gain>
+         <d_gain>2.0</d_gain>
+      </plugin>
+      <plugin filename="gz-sim-joint-position-controller-system"
+               name="gz::sim::systems::JointPositionController">
+         <joint_name>foot_right_joint</joint_name>
+         <topic>/foot_right_joint/cmd</topic>
+         <p_gain>20</p_gain>
+         <i_gain>0</i_gain>
+         <d_gain>2.0</d_gain>
+      </plugin>
+      <plugin filename="gz-sim-joint-position-controller-system"
+               name="gz::sim::systems::JointPositionController">
+         <joint_name>foot_left_joint</joint_name>
+         <topic>/foot_left_joint/cmd</topic>
+         <p_gain>20</p_gain>
+         <i_gain>0</i_gain>
+         <d_gain>2.0</d_gain>
+      </plugin>
+   </gazebo>
+   <!-- Fricção nos pés -->
+   <gazebo reference="FootRight_1">
+   <collision>
+      <surface>
+         <friction>
+         <ode>
+            <mu>10.0</mu>
+            <mu2>10.0</mu2>
+         </ode>
+         </friction>
+      </surface>
+   </collision>
+   </gazebo>
+   <gazebo reference="FootLeft_1">
+   <collision>
+      <surface>
+         <friction>
+         <ode>
+            <mu>10.0</mu>
+            <mu2>10.0</mu2>
+         </ode>
+         </friction>
+      </surface>
+   </collision>
+   </gazebo>
+   <!-- Damping nas juntas para evitar colapso -->
+   <gazebo reference="leg_right_joint">
+   <implicitSpringDamper>true</implicitSpringDamper>
+   <dynamics damping="0.5" friction="0.1"/>
+   </gazebo>
+   <gazebo reference="leg_left_joint">
+   <implicitSpringDamper>true</implicitSpringDamper>
+   <dynamics damping="0.5" friction="0.1"/>
+   </gazebo>
+   <gazebo reference="foot_right_joint">
+   <implicitSpringDamper>true</implicitSpringDamper>
+   <dynamics damping="0.5" friction="0.1"/>
+   </gazebo>
+   <gazebo reference="foot_left_joint">
+   <implicitSpringDamper>true</implicitSpringDamper>
+   <dynamics damping="0.5" friction="0.1"/>
+   </gazebo>
+      <!-- Ancora temporária ao mundo para spawn estável -->
+   <!--<link name="world"/>
+   <joint name="world_fixed" type="fixed">
+      <parent link="world"/>
+      <child link="base_link"/>
+   </joint>
+   -->
 </robot>
