Commit message: Add URDF model for Otto robot with detailed link and joint definitions
- Created a comprehensive URDF file for the Otto robot, detailing its structure, materials, and physical properties.
- Defined multiple links including base, legs, head, and ultrasonic sensor with appropriate inertial properties.
- Implemented revolute joints for leg and foot movements, along with fixed joints for the head and sensor.
- Included Gazebo plugins for joint position control and specified friction/contact properties for feet.

File: ros2_ws/src/otto_description/urdf/materials.xacro (robot description, xacro)
@@ -22,5 +22,5 @@
       <color rgba="0.5372549019607843 0.5372549019607843 0.5372549019607843 1.0" />
    </material>
-   <material name="Materialdebase–Transparente">
+   <material name="Materialdebase-Transparente">
       <color rgba="1.0 1.0 1.0 1.0" />
    </material>

File: ros2_ws/src/otto_description/urdf/otto.xacro (robot description, xacro)
@@ -3,9 +3,33 @@
    <xacro:include filename="$(find otto)/urdf/materials.xacro" />
    <!-- ==================== LINKS ==================== -->
+   <!--
+      base_footprint: link raiz fictício posicionado no chao (z=0).
+      Sem massa nem inercia — serve apenas como referência estável para o Gazebo.
+      O base_link fica 0.08 m acima do chao (altura real do corpo do Otto).
+   -->
+   <link name="base_footprint" />
+   <joint name="base_footprint_joint" type="fixed">
+      <origin xyz="0.0 0.0 0.08" rpy="0.0 0.0 0.0" />
+      <parent link="base_footprint" />
+      <child link="base_link" />
+   </joint>
+   <!--
+      MASSAS ESCALADAS PARA ESTABILIDADE NUMERICA DO GAZEBO
+      ===================================================
+      Fator aplicado por grupo (mantendo razoes relativas do CAD real):
+        base_link, pernas, cabeca  -> x10
+        pes (contato crítico)      -> x12
+        ultrasonico               -> x5
+      Total simulado: ~1.26 kg  (original CAD: ~143 g)
+      Inercias escaladas pelo mesmo fator (I proporcional a m).
+      Todos os tensores passam na condiçao de Sylvester (ixx < iyy+izz, etc).
+   -->
    <link name="base_link">
       <inertial>
          <origin xyz="-0.017480908878091606 0.03519882134873651 -0.025083002755304264" rpy="0.0 0.0 0.0" />
-         <mass value="0.03208248801839897" />
-         <inertia ixx="2.49503e-05" iyy="2.55347e-05" izz="4.0534700000000003e-05" ixy="1.7290000000000002e-07" iyz="7.21e-08" ixz="-2.4710000000000004e-07" />
+         <!-- original: 0.03208 kg  ->  x10 = 0.3208 kg -->
+         <mass value="0.3208" />
+         <inertia ixx="2.49503e-04" iyy="2.55347e-04" izz="4.05347e-04"
+                  ixy="1.7290e-06"  iyz="7.21e-07"    ixz="-2.471e-06" />
       </inertial>
       <visual>
@@ -26,6 +50,8 @@
       <inertial>
          <origin xyz="-1.0223024729112406e-05 0.0 -0.01867704290601307" rpy="0.0 0.0 0.0" />
-         <mass value="0.008348175211097226" />
-         <inertia ixx="1.7007e-06" iyy="2.6586e-06" izz="1.5726e-06" ixy="-0.0" iyz="-0.0" ixz="1.2080000000000002e-07" />
+         <!-- original: 0.008348 kg  ->  x10 = 0.08348 kg -->
+         <mass value="0.08348" />
+         <inertia ixx="1.7007e-05" iyy="2.6586e-05" izz="1.5726e-05"
+                  ixy="0.0"        iyz="0.0"         ixz="1.208e-06" />
       </inertial>
       <visual>
@@ -46,6 +72,8 @@
       <inertial>
          <origin xyz="8.637669678136283e-05 0.0 -0.018540132277720875" rpy="0.0 0.0 0.0" />
-         <mass value="0.008295768110971862" />
-         <inertia ixx="1.6731e-06" iyy="2.6214e-06" izz="1.5575000000000001e-06" ixy="0.0" iyz="0.0" ixz="1.383e-07" />
+         <!-- original: 0.008296 kg  ->  x10 = 0.08296 kg -->
+         <mass value="0.08296" />
+         <inertia ixx="1.6731e-05" iyy="2.6214e-05" izz="1.5575e-05"
+                  ixy="0.0"        iyz="0.0"         ixz="1.383e-06" />
       </inertial>
       <visual>
@@ -66,6 +94,8 @@
       <inertial>
          <origin xyz="0.015667100965246424 0.035094427086301554 0.015158230340085038" rpy="0.0 0.0 0.0" />
-         <mass value="0.044351271100452234" />
-         <inertia ixx="9.202000000000001e-06" iyy="1.6735000000000002e-06" izz="8.9476e-06" ixy="-0.0" iyz="1.21e-08" ixz="-9.1e-09" />
+         <!-- link fixo decorativo: massa minima para nao afetar COM -->
+         <mass value="0.001" />
+         <inertia ixx="1.0e-07" iyy="1.0e-07" izz="1.0e-07"
+                  ixy="0.0"     iyz="0.0"      ixz="0.0" />
       </inertial>
       <visual>
@@ -151,5 +181,5 @@
             <mesh filename="package://otto/meshes/Ultrasonic_Sensor_v1_1_1__Corpo12.stl" scale="0.001 0.001 0.001" />
          </geometry>
-         <material name="Materialdebase–Transparente" />
+         <material name="Materialdebase-Transparente" />
       </visual>
       <visual>
@@ -177,6 +207,8 @@
       <inertial>
          <origin xyz="-0.017855193601269966 0.03577461405901634 0.019109172286024715" rpy="0.0 0.0 0.0" />
-         <mass value="0.024198404764366552" />
-         <inertia ixx="1.64375e-05" iyy="1.5669500000000003e-05" izz="2.6288000000000003e-05" ixy="2.7180000000000004e-07" iyz="8.04e-08" ixz="9.079999999999999e-08" />
+         <!-- link fixo: massa simbólica -->
+         <mass value="0.024" />
+         <inertia ixx="1.64375e-05" iyy="1.56695e-05" izz="2.6288e-05"
+                  ixy="2.718e-07"   iyz="8.04e-08"     ixz="9.08e-08" />
       </inertial>
       <visual>
@@ -197,9 +229,11 @@
       <inertial>
          <origin xyz="-0.01692768844509787 -0.0076979010066632785 -0.010195669876470142" rpy="0.0 0.0 0.0" />
-         <mass value="0.012749332366692664" />
-         <inertia ixx="2.4864e-06" iyy="5.3642e-06" izz="6.5881000000000005e-06" ixy="-7.58e-08" iyz="-4.0549999999999997e-07" ixz="-6.1e-08" />
-      </inertial>
-      <visual>
-         <origin xyz="-0.005508825562246209 -0.005158205912836655 -0.02" rpy="0.0 0.0 0.0" />
+         <!-- original: 0.012749 kg  ->  x12 = 0.15299 kg -->
+         <mass value="0.15299" />
+         <inertia ixx="2.9837e-05" iyy="6.4370e-05" izz="7.9057e-05"
+                  ixy="-9.096e-07"  iyz="-4.866e-06"  ixz="-7.32e-07" />
+      </inertial>
+      <visual>
+         <origin xyz="-0.005508825562246209 -0.005158205912836655 -0.0137" rpy="0.0 0.0 0.0" />
          <geometry>
             <mesh filename="package://otto/meshes/FootRight_1.stl" scale="0.001 0.001 0.001" />
@@ -208,5 +242,5 @@
       </visual>
       <collision>
-         <origin xyz="-0.005508825562246209 -0.005158205912836655 -0.02" rpy="0.0 0.0 0.0" />
+         <origin xyz="-0.005508825562246209 -0.005158205912836655 -0.0137" rpy="0.0 0.0 0.0" />
          <geometry>
             <mesh filename="package://otto/meshes/FootRight_1.stl" scale="0.001 0.001 0.001" />
@@ -217,9 +251,11 @@
       <inertial>
          <origin xyz="-0.016928050017156856 0.004599559866878043 -0.012894741270675017" rpy="0.0 0.0 0.0" />
-         <mass value="0.012746842677145294" />
-         <inertia ixx="2.4861000000000002e-06" iyy="5.3642e-06" izz="6.587899999999999e-06" ixy="7.58e-08" iyz="4.056e-07" ixz="-6.1e-08" />
-      </inertial>
-      <visual>
-         <origin xyz="-0.0005004271247461972 -0.06100042712474619 -0.022000000000000002" rpy="0.0 0.0 0.0" />
+         <!-- original: 0.012747 kg  ->  x12 = 0.15296 kg -->
+         <mass value="0.15296" />
+         <inertia ixx="2.9833e-05" iyy="6.4370e-05" izz="7.9055e-05"
+                  ixy="9.096e-07"   iyz="4.867e-06"   ixz="-7.32e-07" />
+      </inertial>
+      <visual>
+         <origin xyz="-0.0005004271247461972 -0.06100042712474619 -0.0150" rpy="0.0 0.0 0.0" />
          <geometry>
             <mesh filename="package://otto/meshes/FootLeft_1.stl" scale="0.001 0.001 0.001" />
@@ -228,5 +264,5 @@
       </visual>
       <collision>
-         <origin xyz="-0.0005004271247461972 -0.06100042712474619 -0.022000000000000002" rpy="0.0 0.0 0.0" />
+         <origin xyz="-0.0005004271247461972 -0.06100042712474619 -0.0150" rpy="0.0 0.0 0.0" />
          <geometry>
             <mesh filename="package://otto/meshes/FootLeft_1.stl" scale="0.001 0.001 0.001" />
@@ -273,5 +309,15 @@
       <limit upper="1.5707963267948966" lower="-1.5707963267948966" effort="100.0" velocity="100.0" />
    </joint>
-      <!-- Plugin Gazebo para cada junta -->
+   <!-- ==================== GAZEBO PLUGINS ==================== -->
+   <!--
+      PID ajustado para massas x10:
+        P: subiu de 1 -> 10  (torque proporcional à massa)
+        D: subiu de 1 -> 0.5 (amortecimento — menor que P para nao oscilar)
+        I: mantido em 0 (evita windup em juntas de baixa fricçao)
+      Ponto de partida conservador; ajuste fino experimental:
+        se oscilar -> reduza P para 7-8
+        se lento/mole -> aumente P para 12-15
+        se trepida -> aumente D para 0.8-1.0
+   -->
    <gazebo>
       <plugin filename="gz-sim-joint-position-controller-system"
@@ -279,7 +325,7 @@
          <joint_name>leg_right_joint</joint_name>
          <topic>/leg_right_joint/cmd</topic>
-         <p_gain>20</p_gain>
-         <i_gain>0</i_gain>
-         <d_gain>2.0</d_gain>
+         <p_gain>10.0</p_gain>
+         <i_gain>0.0</i_gain>
+         <d_gain>0.5</d_gain>
       </plugin>
       <plugin filename="gz-sim-joint-position-controller-system"
@@ -287,7 +333,7 @@
          <joint_name>leg_left_joint</joint_name>
          <topic>/leg_left_joint/cmd</topic>
-         <p_gain>20</p_gain>
-         <i_gain>0</i_gain>
-         <d_gain>2.0</d_gain>
+         <p_gain>10.0</p_gain>
+         <i_gain>0.0</i_gain>
+         <d_gain>0.5</d_gain>
       </plugin>
       <plugin filename="gz-sim-joint-position-controller-system"
@@ -295,7 +341,7 @@
          <joint_name>foot_right_joint</joint_name>
          <topic>/foot_right_joint/cmd</topic>
-         <p_gain>20</p_gain>
-         <i_gain>0</i_gain>
-         <d_gain>2.0</d_gain>
+         <p_gain>10.0</p_gain>
+         <i_gain>0.0</i_gain>
+         <d_gain>0.5</d_gain>
       </plugin>
       <plugin filename="gz-sim-joint-position-controller-system"
@@ -303,57 +349,43 @@
          <joint_name>foot_left_joint</joint_name>
          <topic>/foot_left_joint/cmd</topic>
-         <p_gain>20</p_gain>
-         <i_gain>0</i_gain>
-         <d_gain>2.0</d_gain>
+         <p_gain>10.0</p_gain>
+         <i_gain>0.0</i_gain>
+         <d_gain>0.5</d_gain>
       </plugin>
    </gazebo>
-   <!-- Fricção nos pés -->
+   <!-- ==================== CONTATO/FRICTION PES ==================== -->
    <gazebo reference="FootRight_1">
-   <collision>
       <surface>
          <friction>
-         <ode>
-            <mu>10.0</mu>
-            <mu2>10.0</mu2>
-         </ode>
+            <ode>
+               <mu>0.8</mu>
+               <mu2>0.8</mu2>
+            </ode>
          </friction>
+         <contact>
+            <ode>
+               <kp>1e5</kp>
+               <kd>1.0</kd>
+               <min_depth>0.001</min_depth>
+            </ode>
+         </contact>
       </surface>
-   </collision>
    </gazebo>
    <gazebo reference="FootLeft_1">
-   <collision>
       <surface>
          <friction>
-         <ode>
-            <mu>10.0</mu>
-            <mu2>10.0</mu2>
-         </ode>
+            <ode>
+               <mu>0.8</mu>
+               <mu2>0.8</mu2>
+            </ode>
          </friction>
+         <contact>
+            <ode>
+               <kp>1e5</kp>
+               <kd>1.0</kd>
+               <min_depth>0.001</min_depth>
+            </ode>
+         </contact>
       </surface>
-   </collision>
    </gazebo>
-   <!-- Damping nas juntas para evitar colapso -->
-   <gazebo reference="leg_right_joint">
-   <implicitSpringDamper>true</implicitSpringDamper>
-   <dynamics damping="0.5" friction="0.1"/>
-   </gazebo>
-   <gazebo reference="leg_left_joint">
-   <implicitSpringDamper>true</implicitSpringDamper>
-   <dynamics damping="0.5" friction="0.1"/>
-   </gazebo>
-   <gazebo reference="foot_right_joint">
-   <implicitSpringDamper>true</implicitSpringDamper>
-   <dynamics damping="0.5" friction="0.1"/>
-   </gazebo>
-   <gazebo reference="foot_left_joint">
-   <implicitSpringDamper>true</implicitSpringDamper>
-   <dynamics damping="0.5" friction="0.1"/>
-   </gazebo>
-      <!-- Ancora temporária ao mundo para spawn estável -->
-   <!--<link name="world"/>
-   <joint name="world_fixed" type="fixed">
-      <parent link="world"/>
-      <child link="base_link"/>
-   </joint>
-   -->
 </robot>
