Commit message: Update URDF for leg and foot links: adjust origins and rotations for accurate positioning

File: ros2_ws/src/otto_description/urdf/otto.urdf (robot description, URDF)
Before this commit: robot otto, 7 links, 6 joints
Joints:
- joint head_joint: origin xyz=0.033 0.0 -0.007 rpy=0 0 0 -> xyz=0.033 0.0 -0.007 rpy=3.14159 0 0

Commit message: Add original Xacro and URDF files for Otto robot description
- Created `otto_Descriptor_Original.xacro` containing detailed robot structure, including links, joints, and materials.
- Introduced `otto_matlab.urdf` generated from the Xacro file, providing a complete URDF representation of the Otto robot with scaled masses and inertias for simulation stability.

File: ros2_ws/src/otto_description/urdf/otto.urdf (robot description, URDF)
Before this commit: robot otto, 8 links, 7 joints
Joints:
- joint foot_right_joint: axis 1.0 0.0 0.0 -> -1.0 0.0 0.0
